File: Design Files/Electrical/yaqubs_keyboard.kicad_pcb (KiCad board)
At the start: 2 copper layers, 386.6 x 120.2 mm, 176 parts

Commit message: init commit
Parts:
- removed the D64 at (418.5, 221.2)
- removed the D71 at (437.6, 202.2)
- removed the S64 at (418.5, 216.2)
- removed the S71 at (437.6, 197.2)
- moved D41 152.1 mm to (263.3, 105.0)
- moved S41 152.1 mm to (263.3, 100.0)
- moved D74 104.5 mm to (368.1, 162.2)
- moved S74 104.5 mm to (368.1, 157.2)
- moved D70 100.3 mm to (339.5, 200.2)
- moved S70 100.3 mm to (339.5, 195.2)
- moved S75 98.1 mm to (358.6, 195.2)
- moved D75 98.1 mm to (358.6, 200.3)
- moved D69 91.2 mm to (349.0, 181.2)
- moved S69 91.2 mm to (349.0, 176.2)
- moved D46 90.9 mm to (253.8, 200.2)
- moved S46 90.9 mm to (253.8, 195.2)
- moved D10 88.5 mm to (54.0, 162.2)
- moved D11 88.5 mm to (54.0, 181.2)
- moved D12 88.5 mm to (54.0, 200.2)
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- renumbered D6 to D1, D9 to D10, D8 to D11, D7 to D12, D18 to D13, D17 to D14, D16 to D15, D15 to D16, D14 to D17, D13 to D18, D24 to D19, D5 to D2, D23 to D20, D22 to D21, D21 to D22, D20 to D23, D19 to D24, D29 to D25, D28 to D26, D26 to D28, D25 to D29, D4 to D3, D87 to D30, D34 to D31, D33 to D32, D32 to D33, D31 to D34, D30 to D35, D39 to D36, D38 to D37, D37 to D38, D36 to D39, D3 to D4, D35 to D40, D88 to D41, D44 to D42, D42 to D44, D41 to D45, D40 to D46, D50 to D47, D49 to D48, D48 to D49, D2 to D5, D47 to D50, D46 to D51, D45 to D52, D56 to D53, D55 to D54, D54 to D55, D53 to D56, D52 to D57, D51 to D58, D62 to D59, D1 to D6, D61 to D60, D60 to D61, D59 to D62, D58 to D63, D57 to D64, D68 to D65, D67 to D66, D66 to D67, D65 to D68, D63 to D69, D12 to D7, D74 to D71, D73 to D72, D72 to D73, D69 to D74, D77 to D75, D80 to D76, D79 to D77, D76 to D79, D11 to D8, D75 to D80, D86 to D81, D85 to D82, D84 to D83, D83 to D84, D82 to D85, D81 to D86, D10 to D9, S6 to S1, S9 to S10, S8 to S11, S7 to S12, S18 to S13, S17 to S14, S16 to S15, S15 to S16, S14 to S17, S13 to S18, S24 to S19, S5 to S2, S23 to S20, S22 to S21, S21 to S22, S20 to S23, S19 to S24, S29 to S25, S28 to S26, S26 to S28, S25 to S29, S4 to S3, S87 to S30, S34 to S31, S33 to S32, S32 to S33, S31 to S34, S30 to S35, S39 to S36, S38 to S37, S37 to S38, S36 to S39, S3 to S4, S35 to S40, S88 to S41, S44 to S42, S42 to S44, S41 to S45, S40 to S46, S50 to S47, S49 to S48, S48 to S49, S2 to S5, S47 to S50, S46 to S51, S45 to S52, S56 to S53, S55 to S54, S54 to S55, S53 to S56, S52 to S57, S51 to S58, S62 to S59, S1 to S6, S61 to S60, S60 to S61, S59 to S62, S58 to S63, S57 to S64, S68 to S65, S67 to S66, S66 to S67, S65 to S68, S63 to S69, S12 to S7, S74 to S71, S73 to S72, S72 to S73, S69 to S74, S77 to S75, S80 to S76, S79 to S77, S76 to S79, S11 to S8, S75 to S80, S86 to S81, S85 to S82, S84 to S83, S83 to S84, S82 to S85, S81 to S86, S10 to S9

Commit message: auto-generated case, pcb with mounting holes.
Parts:
- added C1: 1u, Capacitor_SMD:C_0805_2012Metric, F.Cu at (-89.0, 68.7)
- added C2: 1u, Capacitor_SMD:C_0805_2012Metric, F.Cu at (-89.0, 71.7)
- added C5: 1u, Capacitor_SMD:C_0805_2012Metric, F.Cu at (-109.5, 79.1)
- added D1: SK6812, LED_SMD:LED_SK6812_PLCC4_5.0x5.0mm_P3.2mm, F.Cu at (8.54, -105.6)
- added D10: 1N4148W, Diode_SMD:D_SOD-123, F.Cu at (7.25, -24.3)
- added D100: SK6812, LED_SMD:LED_SK6812MINI_PLCC4_3.5x3.5mm_P1.75mm, F.Cu at (42.2, -59.2)
- added D101: 1N4148W, Diode_SMD:D_SOD-123, F.Cu at (30.4, -27.7)
- added D102: 1N4148W, Diode_SMD:D_SOD-123, F.Cu at (30.4, -24.3)
- added D103: 1N4148W, Diode_SMD:D_SOD-123, F.Cu at (30.4, -21.0)
- added D104: 1N4148W, Diode_SMD:D_SOD-123, F.Cu at (30.4, -17.6)
- added D105: 1N4148W, Diode_SMD:D_SOD-123, F.Cu at (30.4, -14.3)
- added D106: 1N4148W, Diode_SMD:D_SOD-123, F.Cu at (30.4, -10.9)
- added D107: SK6812, LED_SMD:LED_SK6812MINI_PLCC4_3.5x3.5mm_P1.75mm, F.Cu at (42.2, -52.6)
- added D108: SK6812, LED_SMD:LED_SK6812MINI_PLCC4_3.5x3.5mm_P1.75mm, F.Cu at (42.2, -46.0)
- added D109: SK6812, LED_SMD:LED_SK6812MINI_PLCC4_3.5x3.5mm_P1.75mm, F.Cu at (42.2, -39.4)
- added D11: 1N4148W, Diode_SMD:D_SOD-123, F.Cu at (7.25, -21.0)
- added D110: SK6812, LED_SMD:LED_SK6812MINI_PLCC4_3.5x3.5mm_P1.75mm, F.Cu at (50.6, -105.6)
- added D111: SK6812, LED_SMD:LED_SK6812MINI_PLCC4_3.5x3.5mm_P1.75mm, F.Cu at (50.6, -98.9)
- added D112: SK6812, LED_SMD:LED_SK6812MINI_PLCC4_3.5x3.5mm_P1.75mm, F.Cu at (50.6, -92.3)
- added D113: 1N4148W, Diode_SMD:D_SOD-123, F.Cu at (30.4, -7.57)
- added D114: 1N4148W, Diode_SMD:D_SOD-123, F.Cu at (30.4, -4.22)
- added D115: 1N4148W, Diode_SMD:D_SOD-123, F.Cu at (30.4, -0.87)
- added D116: 1N4148W, Diode_SMD:D_SOD-123, F.Cu at (36.2, -34.4)
- added D117: 1N4148W, Diode_SMD:D_SOD-123, F.Cu at (36.2, -31.0)
- added D118: 1N4148W, Diode_SMD:D_SOD-123, F.Cu at (36.2, -27.7)
- added D119: SK6812, LED_SMD:LED_SK6812MINI_PLCC4_3.5x3.5mm_P1.75mm, F.Cu at (50.6, -85.7)
- added D12: 1N4148W, Diode_SMD:D_SOD-123, F.Cu at (7.25, -17.6)
- added D120: SK6812, LED_SMD:LED_SK6812MINI_PLCC4_3.5x3.5mm_P1.75mm, F.Cu at (50.6, -79.1)
- added D121: SK6812, LED_SMD:LED_SK6812MINI_PLCC4_3.5x3.5mm_P1.75mm, F.Cu at (50.6, -72.5)
- added D122: SK6812, LED_SMD:LED_SK6812MINI_PLCC4_3.5x3.5mm_P1.75mm, F.Cu at (50.6, -65.8)
- added D123: SK6812, LED_SMD:LED_SK6812MINI_PLCC4_3.5x3.5mm_P1.75mm, F.Cu at (50.6, -59.2)
- added D124: SK6812, LED_SMD:LED_SK6812MINI_PLCC4_3.5x3.5mm_P1.75mm, F.Cu at (50.6, -52.6)
- added D125: 1N4148W, Diode_SMD:D_SOD-123, F.Cu at (36.2, -24.3)
- added D126: 1N4148W, Diode_SMD:D_SOD-123, F.Cu at (36.2, -21.0)
- added D127: 1N4148W, Diode_SMD:D_SOD-123, F.Cu at (36.2, -17.6)
- added D128: 1N4148W, Diode_SMD:D_SOD-123, F.Cu at (36.2, -14.3)
- added D129: 1N4148W, Diode_SMD:D_SOD-123, F.Cu at (36.2, -10.9)
- added D13: SK6812, LED_SMD:LED_SK6812_PLCC4_5.0x5.0mm_P3.2mm, F.Cu at (8.54, -65.8)
- added D130: 1N4148W, Diode_SMD:D_SOD-123, F.Cu at (36.2, -7.57)
- added D131: SK6812, LED_SMD:LED_SK6812MINI_PLCC4_3.5x3.5mm_P1.75mm, F.Cu at (50.6, -46.0)
- added D132: SK6812, LED_SMD:LED_SK6812MINI_PLCC4_3.5x3.5mm_P1.75mm, F.Cu at (50.6, -39.4)
- added D133: SK6812, LED_SMD:LED_SK6812MINI_PLCC4_3.5x3.5mm_P1.75mm, F.Cu at (59.1, -105.6)
- added D134: SK6812, LED_SMD:LED_SK6812MINI_PLCC4_3.5x3.5mm_P1.75mm, F.Cu at (59.1, -98.9)
- added D135: SK6812, LED_SMD:LED_SK6812MINI_PLCC4_3.5x3.5mm_P1.75mm, F.Cu at (59.1, -92.3)
- added D136: SK6812, LED_SMD:LED_SK6812MINI_PLCC4_3.5x3.5mm_P1.75mm, F.Cu at (59.1, -85.7)
- added D137: 1N4148W, Diode_SMD:D_SOD-123, F.Cu at (36.2, -4.22)
- added D138: 1N4148W, Diode_SMD:D_SOD-123, F.Cu at (36.2, -0.87)
- added D139: 1N4148W, Diode_SMD:D_SOD-123, F.Cu at (42.0, -34.4)
- added D14: SK6812, LED_SMD:LED_SK6812_PLCC4_5.0x5.0mm_P3.2mm, F.Cu at (8.54, -59.2)
- added D140: 1N4148W, Diode_SMD:D_SOD-123, F.Cu at (42.0, -31.0)
- added D141: 1N4148W, Diode_SMD:D_SOD-123, F.Cu at (42.0, -27.7)
- added D142: 1N4148W, Diode_SMD:D_SOD-123, F.Cu at (42.0, -24.3)
- added D143: SK6812, LED_SMD:LED_SK6812MINI_PLCC4_3.5x3.5mm_P1.75mm, F.Cu at (59.1, -79.1)
- added D144: SK6812, LED_SMD:LED_SK6812MINI_PLCC4_3.5x3.5mm_P1.75mm, F.Cu at (59.1, -72.5)
- added D145: SK6812, LED_SMD:LED_SK6812MINI_PLCC4_3.5x3.5mm_P1.75mm, F.Cu at (59.1, -65.8)
- added D146: SK6812, LED_SMD:LED_SK6812MINI_PLCC4_3.5x3.5mm_P1.75mm, F.Cu at (59.1, -59.2)
- added D147: SK6812, LED_SMD:LED_SK6812MINI_PLCC4_3.5x3.5mm_P1.75mm, F.Cu at (59.1, -52.6)
- added D148: 1N4148W, Diode_SMD:D_SOD-123, F.Cu at (42.0, -21.0)
- added D149: 1N4148W, Diode_SMD:D_SOD-123, F.Cu at (42.0, -17.6)
- added D15: SK6812, LED_SMD:LED_SK6812_PLCC4_5.0x5.0mm_P3.2mm, F.Cu at (8.54, -52.6)
- added D150: 1N4148W, Diode_SMD:D_SOD-123, F.Cu at (42.0, -14.3)
- added D151: 1N4148W, Diode_SMD:D_SOD-123, F.Cu at (42.0, -10.9)
- added D152: 1N4148W, Diode_SMD:D_SOD-123, F.Cu at (42.0, -7.57)
- added D153: SK6812, LED_SMD:LED_SK6812MINI_PLCC4_3.5x3.5mm_P1.75mm, F.Cu at (59.1, -46.0)
- added D154: SK6812, LED_SMD:LED_SK6812MINI_PLCC4_3.5x3.5mm_P1.75mm, F.Cu at (59.1, -39.4)
- added D155: SK6812, LED_SMD:LED_SK6812MINI_PLCC4_3.5x3.5mm_P1.75mm, F.Cu at (67.5, -105.6)
- added D156: SK6812, LED_SMD:LED_SK6812MINI_PLCC4_3.5x3.5mm_P1.75mm, F.Cu at (67.5, -98.9)
- added D157: SK6812, LED_SMD:LED_SK6812MINI_PLCC4_3.5x3.5mm_P1.75mm, F.Cu at (67.5, -92.3)
- added D158: 1N4148W, Diode_SMD:D_SOD-123, F.Cu at (42.0, -4.22)
- added D159: 1N4148W, Diode_SMD:D_SOD-123, F.Cu at (42.0, -0.87)
- added D16: SK6812, LED_SMD:LED_SK6812_PLCC4_5.0x5.0mm_P3.2mm, F.Cu at (8.54, -46.0)
- added D160: 1N4148W, Diode_SMD:D_SOD-123, F.Cu at (47.8, -34.4)
- added D161: 1N4148W, Diode_SMD:D_SOD-123, F.Cu at (47.8, -31.0)
- added D162: 1N4148W, Diode_SMD:D_SOD-123, F.Cu at (47.8, -27.7)
- added D163: SK6812, LED_SMD:LED_SK6812MINI_PLCC4_3.5x3.5mm_P1.75mm, F.Cu at (67.5, -85.7)
- added D164: SK6812, LED_SMD:LED_SK6812MINI_PLCC4_3.5x3.5mm_P1.75mm, F.Cu at (67.5, -79.1)
- added D165: SK6812, LED_SMD:LED_SK6812MINI_PLCC4_3.5x3.5mm_P1.75mm, F.Cu at (67.5, -72.5)
- added D166: SK6812, LED_SMD:LED_SK6812MINI_PLCC4_3.5x3.5mm_P1.75mm, F.Cu at (67.5, -65.8)
- added D167: SK6812, LED_SMD:LED_SK6812MINI_PLCC4_3.5x3.5mm_P1.75mm, F.Cu at (67.5, -59.2)
- added D168: SK6812, LED_SMD:LED_SK6812MINI_PLCC4_3.5x3.5mm_P1.75mm, F.Cu at (67.5, -52.6)
- added D169: 1N4148W, Diode_SMD:D_SOD-123, F.Cu at (47.8, -24.3)
- added D17: SK6812, LED_SMD:LED_SK6812_PLCC4_5.0x5.0mm_P3.2mm, F.Cu at (8.54, -39.4)
- added D170: 1N4148W, Diode_SMD:D_SOD-123, F.Cu at (47.8, -21.0)
- added D171: 1N4148W, Diode_SMD:D_SOD-123, F.Cu at (47.8, -17.6)
- added D172: 1N4148W, Diode_SMD:D_SOD-123, F.Cu at (47.8, -14.3)
- added D173: 1N4148W, Diode_SMD:D_SOD-123, F.Cu at (47.8, -10.9)
- added D174: 1N4148W, Diode_SMD:D_SOD-123, F.Cu at (47.8, -7.57)
- added D18: SK6812, LED_SMD:LED_SK6812_PLCC4_5.0x5.0mm_P3.2mm, F.Cu at (17.0, -105.6)
- added D19: 1N4148W, Diode_SMD:D_SOD-123, F.Cu at (7.25, -14.3)
- added D2: SK6812, LED_SMD:LED_SK6812_PLCC4_5.0x5.0mm_P3.2mm, F.Cu at (8.54, -98.9)
- added D20: 1N4148W, Diode_SMD:D_SOD-123, F.Cu at (7.25, -10.9)
- added D21: 1N4148W, Diode_SMD:D_SOD-123, F.Cu at (7.25, -7.57)
- added D22: 1N4148W, Diode_SMD:D_SOD-123, F.Cu at (7.25, -4.22)
- added D23: 1N4148W, Diode_SMD:D_SOD-123, F.Cu at (7.25, -0.87)
- added D24: 1N4148W, Diode_SMD:D_SOD-123, F.Cu at (13.1, -34.4)
- added D25: SK6812, LED_SMD:LED_SK6812MINI_PLCC4_3.5x3.5mm_P1.75mm, F.Cu at (17.0, -98.9)
- added D26: SK6812, LED_SMD:LED_SK6812MINI_PLCC4_3.5x3.5mm_P1.75mm, F.Cu at (17.0, -92.3)
- added D27: SK6812, LED_SMD:LED_SK6812MINI_PLCC4_3.5x3.5mm_P1.75mm, F.Cu at (17.0, -85.7)
- added D28: SK6812, LED_SMD:LED_SK6812MINI_PLCC4_3.5x3.5mm_P1.75mm, F.Cu at (17.0, -79.1)
- added D29: SK6812, LED_SMD:LED_SK6812MINI_PLCC4_3.5x3.5mm_P1.75mm, F.Cu at (17.0, -72.5)
- added D3: SK6812, LED_SMD:LED_SK6812_PLCC4_5.0x5.0mm_P3.2mm, F.Cu at (8.54, -92.3)
- added D30: SK6812, LED_SMD:LED_SK6812MINI_PLCC4_3.5x3.5mm_P1.75mm, F.Cu at (17.0, -65.8)
- added D31: 1N4148W, Diode_SMD:D_SOD-123, F.Cu at (13.1, -31.0)
- added D32: 1N4148W, Diode_SMD:D_SOD-123, F.Cu at (13.1, -27.7)
- added D33: 1N4148W, Diode_SMD:D_SOD-123, F.Cu at (13.1, -24.3)
- added D34: 1N4148W, Diode_SMD:D_SOD-123, F.Cu at (13.1, -21.0)
- added D35: 1N4148W, Diode_SMD:D_SOD-123, F.Cu at (13.1, -17.6)
- added D36: 1N4148W, Diode_SMD:D_SOD-123, F.Cu at (13.1, -14.3)
- added D37: SK6812, LED_SMD:LED_SK6812MINI_PLCC4_3.5x3.5mm_P1.75mm, F.Cu at (17.0, -59.2)
- added D38: SK6812, LED_SMD:LED_SK6812MINI_PLCC4_3.5x3.5mm_P1.75mm, F.Cu at (17.0, -52.6)
- added D39: SK6812, LED_SMD:LED_SK6812MINI_PLCC4_3.5x3.5mm_P1.75mm, F.Cu at (17.0, -46.0)
- added D4: SK6812, LED_SMD:LED_SK6812_PLCC4_5.0x5.0mm_P3.2mm, F.Cu at (8.54, -85.7)
- added D40: SK6812, LED_SMD:LED_SK6812MINI_PLCC4_3.5x3.5mm_P1.75mm, F.Cu at (17.0, -39.4)
- added D41: SK6812, LED_SMD:LED_SK6812MINI_PLCC4_3.5x3.5mm_P1.75mm, F.Cu at (25.4, -105.6)
- added D42: SK6812, LED_SMD:LED_SK6812MINI_PLCC4_3.5x3.5mm_P1.75mm, F.Cu at (25.4, -98.9)
- added D43: 1N4148W, Diode_SMD:D_SOD-123, F.Cu at (13.1, -10.9)
- added D44: 1N4148W, Diode_SMD:D_SOD-123, F.Cu at (13.1, -7.57)
- added D45: 1N4148W, Diode_SMD:D_SOD-123, F.Cu at (13.1, -4.22)
- added D46: 1N4148W, Diode_SMD:D_SOD-123, F.Cu at (13.1, -0.87)
- added D47: 1N4148W, Diode_SMD:D_SOD-123, F.Cu at (18.8, -34.4)
- added D48: 1N4148W, Diode_SMD:D_SOD-123, F.Cu at (18.8, -31.0)
- added D49: SK6812, LED_SMD:LED_SK6812MINI_PLCC4_3.5x3.5mm_P1.75mm, F.Cu at (25.4, -92.3)
- added D5: SK6812, LED_SMD:LED_SK6812_PLCC4_5.0x5.0mm_P3.2mm, F.Cu at (8.54, -79.1)
- added D50: SK6812, LED_SMD:LED_SK6812MINI_PLCC4_3.5x3.5mm_P1.75mm, F.Cu at (25.4, -85.7)
- added D51: SK6812, LED_SMD:LED_SK6812MINI_PLCC4_3.5x3.5mm_P1.75mm, F.Cu at (25.4, -79.1)
- added D52: SK6812, LED_SMD:LED_SK6812MINI_PLCC4_3.5x3.5mm_P1.75mm, F.Cu at (25.4, -72.5)
- added D53: SK6812, LED_SMD:LED_SK6812MINI_PLCC4_3.5x3.5mm_P1.75mm, F.Cu at (25.4, -65.8)
- added D54: SK6812, LED_SMD:LED_SK6812MINI_PLCC4_3.5x3.5mm_P1.75mm, F.Cu at (25.4, -59.2)
- added D55: 1N4148W, Diode_SMD:D_SOD-123, F.Cu at (18.8, -27.7)
- added D56: 1N4148W, Diode_SMD:D_SOD-123, F.Cu at (18.8, -24.3)
- added D57: 1N4148W, Diode_SMD:D_SOD-123, F.Cu at (18.8, -21.0)
- added D58: 1N4148W, Diode_SMD:D_SOD-123, F.Cu at (18.8, -17.6)
- added D59: 1N4148W, Diode_SMD:D_SOD-123, F.Cu at (18.8, -14.3)
- added D6: SK6812, LED_SMD:LED_SK6812_PLCC4_5.0x5.0mm_P3.2mm, F.Cu at (8.54, -72.5)
- added D60: 1N4148W, Diode_SMD:D_SOD-123, F.Cu at (18.8, -10.9)
- added D61: SK6812, LED_SMD:LED_SK6812MINI_PLCC4_3.5x3.5mm_P1.75mm, F.Cu at (25.4, -52.6)
- added D62: SK6812, LED_SMD:LED_SK6812MINI_PLCC4_3.5x3.5mm_P1.75mm, F.Cu at (25.4, -46.0)
- added D63: SK6812, LED_SMD:LED_SK6812MINI_PLCC4_3.5x3.5mm_P1.75mm, F.Cu at (25.4, -39.4)
- added D64: SK6812, LED_SMD:LED_SK6812MINI_PLCC4_3.5x3.5mm_P1.75mm, F.Cu at (33.8, -105.6)
- added D65: SK6812, LED_SMD:LED_SK6812MINI_PLCC4_3.5x3.5mm_P1.75mm, F.Cu at (33.8, -98.9)
- added D66: 1N4148W, Diode_SMD:D_SOD-123, F.Cu at (18.8, -7.57)
- added D67: 1N4148W, Diode_SMD:D_SOD-123, F.Cu at (18.8, -4.22)
- added D68: 1N4148W, Diode_SMD:D_SOD-123, F.Cu at (18.8, -0.87)
- added D69: 1N4148W, Diode_SMD:D_SOD-123, F.Cu at (24.6, -34.4)
- added D7: 1N4148W, Diode_SMD:D_SOD-123, F.Cu at (7.25, -34.4)
- added D70: 1N4148W, Diode_SMD:D_SOD-123, F.Cu at (24.6, -31.0)
- added D71: SK6812, LED_SMD:LED_SK6812MINI_PLCC4_3.5x3.5mm_P1.75mm, F.Cu at (33.8, -92.3)
- added D72: SK6812, LED_SMD:LED_SK6812MINI_PLCC4_3.5x3.5mm_P1.75mm, F.Cu at (33.8, -85.7)
- added D73: SK6812, LED_SMD:LED_SK6812MINI_PLCC4_3.5x3.5mm_P1.75mm, F.Cu at (33.8, -79.1)
- added D74: SK6812, LED_SMD:LED_SK6812MINI_PLCC4_3.5x3.5mm_P1.75mm, F.Cu at (33.8, -72.5)
- added D75: SK6812, LED_SMD:LED_SK6812MINI_PLCC4_3.5x3.5mm_P1.75mm, F.Cu at (33.8, -65.8)
- added D76: 1N4148W, Diode_SMD:D_SOD-123, F.Cu at (24.6, -27.7)
- added D77: 1N4148W, Diode_SMD:D_SOD-123, F.Cu at (24.6, -24.3)
- added D78: 1N4148W, Diode_SMD:D_SOD-123, F.Cu at (24.6, -21.0)
- added D79: 1N4148W, Diode_SMD:D_SOD-123, F.Cu at (24.6, -17.6)
- added D8: 1N4148W, Diode_SMD:D_SOD-123, F.Cu at (7.25, -31.0)
- added D80: 1N4148W, Diode_SMD:D_SOD-123, F.Cu at (24.6, -14.3)
- added D81: SK6812, LED_SMD:LED_SK6812MINI_PLCC4_3.5x3.5mm_P1.75mm, F.Cu at (33.8, -59.2)
- added D82: SK6812, LED_SMD:LED_SK6812MINI_PLCC4_3.5x3.5mm_P1.75mm, F.Cu at (33.8, -52.6)
- added D83: SK6812, LED_SMD:LED_SK6812MINI_PLCC4_3.5x3.5mm_P1.75mm, F.Cu at (33.8, -46.0)
- added D84: SK6812, LED_SMD:LED_SK6812MINI_PLCC4_3.5x3.5mm_P1.75mm, F.Cu at (33.8, -39.4)
- added D85: SK6812, LED_SMD:LED_SK6812MINI_PLCC4_3.5x3.5mm_P1.75mm, F.Cu at (42.2, -105.6)
- added D86: SK6812, LED_SMD:LED_SK6812MINI_PLCC4_3.5x3.5mm_P1.75mm, F.Cu at (42.2, -98.9)
- added D87: 1N4148W, Diode_SMD:D_SOD-123, F.Cu at (24.6, -10.9)
- added D88: 1N4148W, Diode_SMD:D_SOD-123, F.Cu at (24.6, -7.57)
- added D9: 1N4148W, Diode_SMD:D_SOD-123, F.Cu at (7.25, -27.7)
- added D91: 1N4148W, Diode_SMD:D_SOD-123, F.Cu at (24.6, -4.22)
- added D92: 1N4148W, Diode_SMD:D_SOD-123, F.Cu at (24.6, -0.87)
- added D93: 1N4148W, Diode_SMD:D_SOD-123, F.Cu at (30.4, -34.4)
- added D94: 1N4148W, Diode_SMD:D_SOD-123, F.Cu at (30.4, -31.0)
- added D95: SK6812, LED_SMD:LED_SK6812MINI_PLCC4_3.5x3.5mm_P1.75mm, F.Cu at (42.2, -92.3)
- added D96: SK6812, LED_SMD:LED_SK6812MINI_PLCC4_3.5x3.5mm_P1.75mm, F.Cu at (42.2, -85.7)
- added D97: SK6812, LED_SMD:LED_SK6812MINI_PLCC4_3.5x3.5mm_P1.75mm, F.Cu at (42.2, -79.1)
- added D98: SK6812, LED_SMD:LED_SK6812MINI_PLCC4_3.5x3.5mm_P1.75mm, F.Cu at (42.2, -72.5)
- added D99: SK6812, LED_SMD:LED_SK6812MINI_PLCC4_3.5x3.5mm_P1.75mm, F.Cu at (42.2, -65.8)
- added FB1: 100Ω @ 100MHz, Resistor_SMD:R_0805_2012Metric, F.Cu at (-84.6, 68.7)
- added J2: OLED Interface, Connector_PinHeader_2.54mm:PinHeader_1x07_P2.54mm_Vertical, F.Cu at (-62.0, 84.2)
- added U1: STM32G474VETx, Package_QFP:LQFP-100_14x14mm_P0.5mm, F.Cu at (186.2, 107.5)
- added U2: AMS1117CD-3.3, Package_TO_SOT_SMD:TO-252-3_TabPin2, F.Cu at (-76.9, 57.2)
- S1, S10, S11, S12, S13, S14, S15, S16, S17, S18, S19, S2, S20, S21, S22, S23, S24, S25, S26, S27, S28, S29, S3, S30, S31, S32, S33, S34, S35, S36, S37, S38, S39, S4, S40, S41, S42, S43, S44, S45, S46, S47, S48, S49, S5, S50, S51, S52, S53, S54, S55, S56, S57, S58, S59, S6, S60, S61, S62, S63, S64, S65, S66, S67, S68, S69, S7, S70, S71, S72, S73, S74, S75, S76, S77, S78, S79, S8, S80, S81, S82, S83, S84, S85, S86, S9: footprint MX -> PCM_Switch_Keyboard_Cherry_MX:SW_Cherry_MX_PCB_1.00u
