File: Design Files/Electrical/yaqubs_keyboard.kicad_sch (KiCad schematic)
At the start: 1 part, among them U1 STM32G474VCTx

Commit message: init commit
Parts:
- removed U1: STM32G474VCTx, Package_QFP:LQFP-100_14x14mm_P0.5mm, symbol MCU_ST_STM32G4:STM32G474VCTx
- added D1, D10, D11, D12, D13, D14, D15, D16, D17, D18, D19, D2, D20, D21, D22, D23, D24, D25, D26, D27, D28, D29, D3, D30, D31, D32, D33, D34, D35, D36, D37, D38, D39, D4, D40, D41, D42, D43, D44, D45, D46, D47, D48, D49, D5, D50, D51, D52, D53, D54, D55, D56, D57, D58, D59, D6, D60, D61, D62, D63, D64, D65, D66, D67, D68, D69, D7, D70, D71, D72, D73, D74, D75, D76, D77, D78, D79, D8, D80, D81, D82, D83, D84, D85, D86, D9: 1N4148W, Diode_SMD:D_SOD-123, symbol Diode:1N4148W
- added D87: SK6812, LED_SMD:LED_SK6812_PLCC4_5.0x5.0mm_P3.2mm, symbol LED:SK6812
- added D89, D90: 3.6 V, symbol Yaqubs_Cool_Parts:ESD321DPYR
- added DS1: OLED-128O064D, Display:OLED-128O064D, symbol Display_Graphic:OLED-128O064D
- added F1: 500 mA, symbol Yaqubs_Cool_Parts:0ZCG0050AF2C
- added FB1: 100Ω @ 100MHz, Resistor_SMD:R_0805_2012Metric, symbol Yaqubs_Cool_Parts:MPZ2012S101AT000
- added J1: USB_C_Receptacle_USB2.0_16P, symbol Connector:USB_C_Receptacle_USB2.0_16P
- added R1, R2: 5.1k, symbol Yaqubs_Cool_Parts:RES_5.1KOHM_0805
- added S1, S10, S11, S12, S13, S14, S15, S16, S17, S18, S19, S2, S20, S21, S22, S23, S24, S25, S26, S27, S28, S29, S3, S30, S31, S32, S33, S34, S35, S36, S37, S38, S39, S4, S40, S41, S42, S43, S44, S45, S46, S47, S48, S49, S5, S50, S51, S52, S53, S54, S55, S56, S57, S58, S59, S6, S60, S61, S62, S63, S64, S65, S66, S67, S68, S69, S7, S70, S71, S72, S73, S74, S75, S76, S77, S78, S79, S8, S80, S81, S82, S83, S84, S85, S86, S9: MX_key, Button_Switch_Keyboard:SW_Cherry_MX_1.00u_PCB, symbol Yaqubs_Cool_Parts:MX_key
- added U1: STM32G474MBTx, Package_QFP:LQFP-80_12x12mm_P0.5mm, symbol MCU_ST_STM32G4:STM32G474MBTx
Connections:
- new net: D62.2 (A), S62.2
- new net: D76.2 (A), S76.2
- new net: D28.2 (A), S28.2
- new net: D74.2 (A), S74.2
- new net: D65.2 (A), S65.2
- new net: D55.2 (A), S55.2
- new net: D61.2 (A), S61.2
- new net: D57.2 (A), S57.2
- new net: D24.2 (A), S24.2
- new net: D54.2 (A), S54.2
- new net: D53.2 (A), S53.2
- new net: D42.2 (A), S42.2
- new net: D81.2 (A), S81.2
- new net: D59.2 (A), S59.2
- new net: D64.2 (A), S64.2
- new net: D73.2 (A), S73.2
- new net: D48.2 (A), S48.2
- new net: D71.2 (A), S71.2
- new net: D33.2 (A), S33.2
- new net: D6.2 (A), S6.2
- new net: D35.2 (A), S35.2
- new net: D34.2 (A), S34.2
- new net: D58.2 (A), S58.2
- new net: D2.2 (A), S2.2
- new net: D36.2 (A), S36.2
- new net: D85.2 (A), S85.2
- new net: D40.2 (A), S40.2
- new net: D66.2 (A), S66.2
- new net: D7.2 (A), S7.2
- new net: D68.2 (A), S68.2
- new net: D69.2 (A), S69.2
- new net: D51.2 (A), S51.2
- new net: D77.2 (A), S77.2
- new net: D14.2 (A), S14.2
- new net: D84.2 (A), S84.2
- new net: D9.2 (A), S9.2
- new net: D82.2 (A), S82.2
- new net: D60.2 (A), S60.2
- new net: D50.2 (A), S50.2
- new net: D86.2 (A), S86.2
- new net: D23.2 (A), S23.2
- new net: D80.2 (A), S80.2
- new net: D11.2 (A), S11.2
- new net: D45.2 (A), S45.2
- new net: D75.2 (A), S75.2
- new net: D70.2 (A), S70.2
- new net: D79.2 (A), S79.2
- new net: D20.2 (A), S20.2
- new net: D27.2 (A), S27.2
- new net: U1.15 (VSS), U1.40 (VSS), U1.50 (VSS), U1.61 (VSS), U1.79 (VSS)
- new net: F1.1, FB1.2
- new net: D52.2 (A), S52.2
- new net: D44.2 (A), S44.2
- new net: D49.2 (A), S49.2
- new net: D18.2 (A), S18.2
- new net: D8.2 (A), S8.2
- new net: D37.2 (A), S37.2
- new net: D56.2 (A), S56.2
- new net: D46.2 (A), S46.2
- new net: D26.2 (A), S26.2
- new net: D22.2 (A), S22.2
- new net: D29.2 (A), S29.2
- new net: D10.2 (A), S10.2
- new net: D16.2 (A), S16.2
- new net: D32.2 (A), S32.2
- new net: J1.B5 (CC2), R2.1
- new net: D1.2 (A), S1.2
- new net: D21.2 (A), S21.2
- new net: D3.2 (A), S3.2
- new net: D43.2 (A), S43.2
- new net: FB1.1, J1.A4 (VBUS), J1.A9 (VBUS), J1.B4 (VBUS), J1.B9 (VBUS)
- new net: D41.2 (A), S41.2
- new net: D38.2 (A), S38.2
- new net: D5.2 (A), S5.2
- new net: D63.2 (A), S63.2
- new net: D4.2 (A), S4.2
- new net: D17.2 (A), S17.2
- new net: D13.2 (A), S13.2
- new net: D25.2 (A), S25.2
- new net: D15.2 (A), S15.2
- new net: D78.2 (A), S78.2
- new net: D72.2 (A), S72.2
- new net: D47.2 (A), S47.2
- new net: J1.A5 (CC1), R1.1
- new net: D67.2 (A), S67.2
- new net: DS1.1 (GND), DS1.30 (GND)
- new net: D30.2 (A), S30.2
- new net: D39.2 (A), S39.2
- new net: D83.2 (A), S83.2
- new net: D31.2 (A), S31.2
- new net: D12.2 (A), S12.2
- new net: D19.2 (A), S19.2
- new net +5V: F1.2
- new net COL0: S1.1, S2.1, S3.1, S4.1, S5.1, S6.1
- new net COL1: S10.1, S11.1, S12.1, S7.1, S8.1, S9.1
- new net COL10: S59.1, S60.1, S61.1, S62.1, S63.1, S64.1
- new net COL11: S65.1, S66.1, S67.1, S68.1, S69.1, S70.1
- new net COL12: S71.1, S72.1, S73.1, S74.1, S75.1
- new net COL13: S76.1, S77.1, S78.1, S79.1, S80.1
- new net COL14: S81.1, S82.1, S83.1, S84.1, S85.1, S86.1
- new net COL2: S13.1, S14.1, S15.1, S16.1, S17.1, S18.1
- new net COL3: S19.1, S20.1, S21.1, S22.1, S23.1, S24.1
- new net COL4: S25.1, S26.1, S27.1, S28.1, S29.1, S30.1
- new net COL5: S31.1, S32.1, S33.1, S34.1, S35.1
- new net COL6: S36.1, S37.1, S38.1, S39.1, S40.1
- new net COL7: S41.1, S42.1, S43.1, S44.1, S45.1, S46.1
- new net COL8: S47.1, S48.1, S49.1, S50.1, S51.1, S52.1
- new net COL9: S53.1, S54.1, S55.1, S56.1, S57.1, S58.1
- new net D+: D89.1 (K), J1.A6 (D+), J1.B6 (D+)
- new net D-: D90.1 (K), J1.A7 (D-), J1.B7 (D-)
- new net GND: D89.2 (A), D90.2 (A), J1.A1 (GND), J1.A12 (GND), J1.B1 (GND), J1.B12 (GND), J1.S1 (SHIELD), R1.2, R2.2
- new net ROW0: D1.1 (K), D13.1 (K), D19.1 (K), D25.1 (K), D31.1 (K), D36.1 (K), D41.1 (K), D47.1 (K), D53.1 (K), D59.1 (K), D65.1 (K), D7.1 (K), D71.1 (K), D76.1 (K), D81.1 (K)
- new net ROW1: D14.1 (K), D2.1 (K), D20.1 (K), D26.1 (K), D32.1 (K), D37.1 (K), D42.1 (K), D48.1 (K), D54.1 (K), D60.1 (K), D66.1 (K), D72.1 (K), D77.1 (K), D8.1 (K), D82.1 (K)
- new net ROW2: D15.1 (K), D21.1 (K), D27.1 (K), D3.1 (K), D33.1 (K), D38.1 (K), D43.1 (K), D49.1 (K), D55.1 (K), D61.1 (K), D67.1 (K), D73.1 (K), D78.1 (K), D83.1 (K), D9.1 (K)
- new net ROW3: D10.1 (K), D16.1 (K), D22.1 (K), D28.1 (K), D34.1 (K), D39.1 (K), D4.1 (K), D44.1 (K), D50.1 (K), D56.1 (K), D62.1 (K), D68.1 (K), D74.1 (K), D79.1 (K), D84.1 (K)
- new net ROW4: D11.1 (K), D17.1 (K), D23.1 (K), D29.1 (K), D35.1 (K), D40.1 (K), D45.1 (K), D5.1 (K), D51.1 (K), D57.1 (K), D63.1 (K), D69.1 (K), D75.1 (K), D80.1 (K), D85.1 (K)
- new net ROW5: D12.1 (K), D18.1 (K), D24.1 (K), D30.1 (K), D46.1 (K), D52.1 (K), D58.1 (K), D6.1 (K), D64.1 (K), D70.1 (K), D86.1 (K)
- no-connect marks 0 -> 2

Commit message: auto-generated case, pcb with mounting holes.
Parts:
- removed D1, D10, D11, D12, D13, D14, D15, D16, D17, D18, D19, D2, D20, D21, D22, D23, D24, D25, D26, D27, D28, D29, D3, D30, D31, D32, D33, D34, D35, D36, D37, D38, D39, D4, D40, D41, D42, D43, D44, D45, D46, D47, D48, D49, D5, D50, D51, D52, D53, D54, D55, D56, D57, D58, D59, D6, D60, D61, D62, D63, D64, D65, D66, D67, D68, D69, D7, D70, D71, D72, D73, D74, D75, D76, D77, D78, D79, D8, D80, D81, D82, D83, D84, D85, D86, D9: 1N4148W, Diode_SMD:D_SOD-123, symbol Diode:1N4148W
- removed D87: SK6812, LED_SMD:LED_SK6812_PLCC4_5.0x5.0mm_P3.2mm, symbol LED:SK6812
- removed D89, D90: 3.6 V, symbol Yaqubs_Cool_Parts:ESD321DPYR
- removed DS1: OLED-128O064D, Display:OLED-128O064D, symbol Display_Graphic:OLED-128O064D
- removed F1: 500 mA, symbol Yaqubs_Cool_Parts:0ZCG0050AF2C
- removed FB1: 100Ω @ 100MHz, Resistor_SMD:R_0805_2012Metric, symbol Yaqubs_Cool_Parts:MPZ2012S101AT000
- removed J1: USB_C_Receptacle_USB2.0_16P, symbol Connector:USB_C_Receptacle_USB2.0_16P
- removed R1, R2: 5.1k, symbol Yaqubs_Cool_Parts:RES_5.1KOHM_0805
- removed S1, S10, S11, S12, S13, S14, S15, S16, S17, S18, S19, S2, S20, S21, S22, S23, S24, S25, S26, S27, S28, S29, S3, S30, S31, S32, S33, S34, S35, S36, S37, S38, S39, S4, S40, S41, S42, S43, S44, S45, S46, S47, S48, S49, S5, S50, S51, S52, S53, S54, S55, S56, S57, S58, S59, S6, S60, S61, S62, S63, S64, S65, S66, S67, S68, S69, S7, S70, S71, S72, S73, S74, S75, S76, S77, S78, S79, S8, S80, S81, S82, S83, S84, S85, S86, S9: MX_key, Button_Switch_Keyboard:SW_Cherry_MX_1.00u_PCB, symbol Yaqubs_Cool_Parts:MX_key
- removed U1: STM32G474MBTx, Package_QFP:LQFP-80_12x12mm_P0.5mm, symbol MCU_ST_STM32G4:STM32G474MBTx
Connections:
- no-connect marks 2 -> 0
Other:
- added sheet Input (input.kicad_sch)
- added sheet LED and Switch Matrices (matrix.kicad_sch)
- added sheet MCU (MCU.kicad_sch)
